File: pcb_layouts/seamonster_smd/seamonster_smd_draft1/seamonster_smd_draft1.brd (EAGLE design)
At the start: 172.5 x 106.5 mm, 78 parts, among them IC1 7805T, IC2 4051D, IC3 4051D, IC4 DG408DY, IC5 4040D, IC6 40106D, IC7 4070D, Q1 THONKICONNNEW, Q2 THONKICONNNEW, Q3 THONKICONNNEW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

Commit message: added new panel drill files for prototype panel
Parts:
- added U$2, U$3, U$4, U$5: T-80-T-SPDT-ON-OFF-ON, MusicThingModular:M9040P
- added VR10, VR11, VR12: (no value), MusicThingModular:9MM_SNAP-IN_POT
- added VR9: 100KΩ, MusicThingModular:9MM_SNAP-IN_POT
Connections:
- new net CCO1: IC6.4, VR9.2
- new net N$46: IC6.3, U$2.2, VR9.1
- new net N$47: CCO1_OUT.P$1_TIP, U1.1, U1.2
- new net N$52: CCO2_OUT.P$1_TIP, U1.6, U1.7
- new net N$53: CCO3_OUT.P$1_TIP, U1.8, U1.9
- new net N$54: CCO4_OUT.P$1_TIP, U1.13, U1.14
- new net N$55: U1.3
- new net N$56: U1.5
- new net N$57: U1.10
- new net N$58: U1.12
- new net N$59: U2.1, U2.2, VCO1_OUT.P$1_TIP
- new net N$60: U2.6, U2.7, VCO2_OUT.P$1_TIP
- new net N$61: COMPLEX_OUT1.P$1_TIP, U2.8, U2.9
- new net N$63: COMPLEX_OUT2.P$1_TIP, U2.13, U2.14
- new net N$67: U2.3
- new net N$68: U2.5
- new net N$69: U2.10
- new net N$70: U2.12
- net GND: now also CCO1_OUT.P$3_SLEEVE, CCO2_OUT.P$3_SLEEVE, CCO3_OUT.P$3_SLEEVE, CCO4_OUT.P$3_SLEEVE, COMPLEX_OUT1.P$3_SLEEVE, COMPLEX_OUT2.P$3_SLEEVE, VCO1_OUT.P$3_SLEEVE, VCO2_OUT.P$3_SLEEVE
Changed lines of the file:
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@@
 <element name="R13" library="SparkFun-Resistors" package="0805" value="" x="-234.95" y="-118.11"/>
 <element name="R14" library="SparkFun-Resistors" package="0805" value="" x="-238.76" y="-118.11"/>
+<element name="U$2" library="MusicThingModular" package="M9040P" value="T-80-T-SPDT-ON-OFF-ON" x="-256.54" y="-100.33"/>
+<element name="U$3" library="MusicThingModular" package="M9040P" value="T-80-T-SPDT-ON-OFF-ON" x="-289.56" y="-100.33"/>
+<element name="U$4" library="MusicThingModular" package="M9040P" value="T-80-T-SPDT-ON-OFF-ON" x="-322.58" y="-100.33"/>
+<element name="U$5" library="MusicThingModular" package="M9040P" value="T-80-T-SPDT-ON-OFF-ON" x="-355.6" y="-100.33"/>
+<element name="VR9" library="MusicThingModular" package="9MM_SNAP-IN_POT" value="100KΩ" x="-350.52" y="-137.16"/>
+<element name="VR10" library="MusicThingModular" package="9MM_SNAP-IN_POT" value="" x="-350.52" y="-168.91"/>
+<element name="VR11" library="MusicThingModular" package="9MM_SNAP-IN_POT" value="" x="-350.52" y="-200.66"/>
+<element name="VR12" library="MusicThingModular" package="9MM_SNAP-IN_POT" value="" x="-350.52" y="-232.41"/>
 </elements>
 <signals>
@@
 <contactref element="Q2" pad="P$3_SLEEVE"/>
 <contactref element="Q1" pad="P$3_SLEEVE"/>
+<contactref element="CCO1_OUT" pad="P$3_SLEEVE"/>
+<contactref element="CCO4_OUT" pad="P$3_SLEEVE"/>
+<contactref element="CCO2_OUT" pad="P$3_SLEEVE"/>
+<contactref element="CCO3_OUT" pad="P$3_SLEEVE"/>
+<contactref element="COMPLEX_OUT2" pad="P$3_SLEEVE"/>
+<contactref element="COMPLEX_OUT1" pad="P$3_SLEEVE"/>
+<contactref element="VCO2_OUT" pad="P$3_SLEEVE"/>
+<contactref element="VCO1_OUT" pad="P$3_SLEEVE"/>
 <wire x1="-205.74" y1="-16.51" x2="-205.74" y2="-35.56" width="0" layer="19" extent="1-1"/>
 <wire x1="-205.74" y1="-54.61" x2="-205.74" y2="-35.56" width="0" layer="19" extent="1-1"/>
@@
 <wire x1="10.16" y1="73.51" x2="29.21" y2="73.51" width="0" layer="19" extent="1-1"/>
 <wire x1="-21.59" y1="2.54" x2="-57.15" y2="14.12" width="0" layer="19" extent="1-1"/>
+<wire x1="7.62" y1="26.82" x2="-21.59" y2="2.54" width="0" layer="19" extent="1-1"/>
+<wire x1="17.78" y1="26.82" x2="7.62" y2="26.82" width="0" layer="19" extent="1-1"/>
+<wire x1="27.94" y1="26.82" x2="17.78" y2="26.82" width="0" layer="19" extent="1-1"/>
+<wire x1="38.1" y1="26.82" x2="27.94" y2="26.82" width="0" layer="19" extent="1-1"/>
+<wire x1="48.26" y1="26.82" x2="38.1" y2="26.82" width="0" layer="19" extent="1-1"/>
+<wire x1="58.42" y1="26.82" x2="48.26" y2="26.82" width="0" layer="19" extent="1-1"/>
+<wire x1="68.58" y1="26.82" x2="58.42" y2="26.82" width="0" layer="19" extent="1-1"/>
+<wire x1="78.74" y1="26.82" x2="68.58" y2="26.82" width="0" layer="19" extent="1-1"/>
 </signal>
 <signal name="VCC">
@@
 <contactref element="R14" pad="2"/>
 </signal>
+<signal name="N$46">
+<contactref element="U$2" pad="2"/>
+<contactref element="IC6" pad="3"/>
+<contactref element="VR9" pad="1"/>
+<wire x1="-256.54" y1="-100.33" x2="-353.02" y2="-144.16" width="0" layer="19" extent="1-1"/>
+<wire x1="-101.6" y1="-3.0734" x2="-256.54" y2="-100.33" width="0" layer="19" extent="1-1"/>
+</signal>
+<signal name="CCO1">
+<contactref element="VR9" pad="2"/>
+<contactref element="IC6" pad="4"/>
+<wire x1="-100.33" y1="-3.0734" x2="-350.52" y2="-144.16" width="0" layer="19" extent="1-1"/>
+</signal>
+<signal name="N$47">
+<contactref element="U1" pad="2"/>
+<contactref element="U1" pad="1"/>
+<contactref element="CCO1_OUT" pad="P$1_TIP"/>
+<wire x1="-87.63" y1="65.98" x2="-86.36" y2="65.98" width="0" layer="19" extent="1-1"/>
+<wire x1="7.62" y1="15.32" x2="-86.36" y2="65.98" width="0" layer="19" extent="1-1"/>
+</signal>
+<signal name="N$52">
+<contactref element="U1" pad="6"/>
+<contactref element="U1" pad="7"/>
+<contactref element="CCO2_OUT" pad="P$1_TIP"/>
+<wire x1="-80.01" y1="65.98" x2="17.78" y2="15.32" width="0" layer="19" extent="1-1"/>
+<wire x1="-81.28" y1="65.98" x2="-80.01" y2="65.98" width="0" layer="19" extent="1-1"/>
+</signal>
+<signal name="N$53">
+<contactref element="U1" pad="9"/>
+<contactref element="U1" pad="8"/>
+<contactref element="CCO3_OUT" pad="P$1_TIP"/>
+<wire x1="-80.01" y1="71.18" x2="27.94" y2="15.32" width="0" layer="19" extent="1-1"/>
+<wire x1="-81.28" y1="71.18" x2="-80.01" y2="71.18" width="0" layer="19" extent="1-1"/>
+</signal>
+<signal name="N$54">
+<contactref element="U1" pad="13"/>
+<contactref element="U1" pad="14"/>
+<contactref element="CCO4_OUT" pad="P$1_TIP"/>
+<wire x1="-86.36" y1="71.18" x2="38.1" y2="15.32" width="0" layer="19" extent="1-1"/>
+<wire x1="-87.63" y1="71.18" x2="-86.36" y2="71.18" width="0" layer="19" extent="1-1"/>
+</signal>
+<signal name="N$55">
+<contactref element="U1" pad="3"/>
+</signal>
+<signal name="N$56">
+<contactref element="U1" pad="5"/>
+</signal>
+<signal name="N$57">
+<contactref element="U1" pad="10"/>
+</signal>
+<signal name="N$58">
+<contactref element="U1" pad="12"/>
+</signal>
+<signal name="N$59">
+<contactref element="U2" pad="2"/>
+<contactref element="U2" pad="1"/>
+<contactref element="VCO1_OUT" pad="P$1_TIP"/>
+<wire x1="-21.59" y1="81.22" x2="48.26" y2="15.32" width="0" layer="19" extent="1-1"/>
+<wire x1="-22.86" y1="81.22" x2="-21.59" y2="81.22" width="0" layer="19" extent="1-1"/>
+</signal>
+<signal name="N$60">
+<contactref element="U2" pad="6"/>
+<contactref element="U2" pad="7"/>
+<contactref element="VCO2_OUT" pad="P$1_TIP"/>
+<wire x1="-15.24" y1="81.22" x2="58.42" y2="15.32" width="0" layer="19" extent="1-1"/>
+<wire x1="-16.51" y1="81.22" x2="-15.24" y2="81.22" width="0" layer="19" extent="1-1"/>
+</signal>
+<signal name="N$61">
+<contactref element="U2" pad="9"/>
+<contactref element="U2" pad="8"/>
+<contactref element="COMPLEX_OUT1" pad="P$1_TIP"/>
+<wire x1="-15.24" y1="86.42" x2="68.58" y2="15.32" width="0" layer="19" extent="1-1"/>
+<wire x1="-16.51" y1="86.42" x2="-15.24" y2="86.42" width="0" layer="19" extent="1-1"/>
+</signal>
+<signal name="N$63">
+<contactref element="U2" pad="13"/>
+<contactref element="U2" pad="14"/>
+<contactref element="COMPLEX_OUT2" pad="P$1_TIP"/>
+<wire x1="-21.59" y1="86.42" x2="78.74" y2="15.32" width="0" layer="19" extent="1-1"/>
+<wire x1="-22.86" y1="86.42" x2="-21.59" y2="86.42" width="0" layer="19" extent="1-1"/>
+</signal>
+<signal name="N$67">
+<contactref element="U2" pad="3"/>
+</signal>
+<signal name="N$68">
+<contactref element="U2" pad="5"/>
+</signal>
+<signal name="N$69">
+<contactref element="U2" pad="10"/>
+</signal>
+<signal name="N$70">
+<contactref element="U2" pad="12"/>
+</signal>
 </signals>
