File: pcb_layouts/seamonster_smd/seamonster_smd_draft1/seamonster_smd_draft1.sch (EAGLE design)
At the start: 78 parts, among them IC1 7805T, IC2 4051D, IC3 4051D, IC4 DG408DY, IC5 4040D, IC6 40106D, IC7 4070D, Q1 THONKICONNNEW, Q2 THONKICONNNEW, Q3 THONKICONNNEW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

Commit message: added new panel drill files for prototype panel
Parts:
- added U$2, U$3, U$4, U$5: T-80-T-SPDT-ON-OFF-ON, MusicThingModular:T-80-T-SPDT-ON-OFF-ON
- added VR10, VR11, VR12: (no value), MusicThingModular:9MM_SNAP-IN_POT_
- added VR9: 100KΩ, MusicThingModular:9MM_SNAP-IN_POT_
Connections:
- new net CCO1: IC6B.O, VR9.S
- new net N$46: IC6B.I, U$2.P, VR9.A
- new net N$47: CCO1_OUT.TIP, U1A.-IN, U1A.OUT
- new net N$52: CCO2_OUT.TIP, U1B.-IN, U1B.OUT
- new net N$53: CCO3_OUT.TIP, U1C.-IN, U1C.OUT
- new net N$54: CCO4_OUT.TIP, U1D.-IN, U1D.OUT
- new net N$55: U1A.+IN
- new net N$56: U1B.+IN
- new net N$57: U1C.+IN
- new net N$58: U1D.+IN
- new net N$59: U2A.-IN, U2A.OUT, VCO1_OUT.TIP
- new net N$60: U2B.-IN, U2B.OUT, VCO2_OUT.TIP
- new net N$61: COMPLEX_OUT1.TIP, U2C.-IN, U2C.OUT
- new net N$63: COMPLEX_OUT2.TIP, U2D.-IN, U2D.OUT
- new net N$67: U2A.+IN
- new net N$68: U2B.+IN
- new net N$69: U2C.+IN
- new net N$70: U2D.+IN
- net GND: now also CCO1_OUT.SLEEVE, CCO2_OUT.SLEEVE, CCO3_OUT.SLEEVE, CCO4_OUT.SLEEVE, COMPLEX_OUT1.SLEEVE, COMPLEX_OUT2.SLEEVE, VCO1_OUT.SLEEVE, VCO2_OUT.SLEEVE
Other:
- moved on the sheet: CCO1_OUT, CCO2_OUT, CCO3_OUT, CCO4_OUT, COMPLEX_OUT1, COMPLEX_OUT2, IC6B, U1A, U1B, U1C, U1D, U2A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
