File: pcb_layouts/seamonster_schematic.sch (EAGLE design)
At the start: 132 parts, among them IC1 7808DT, IC2 4051D, IC3 4051D, IC4 DG408DY, IC5 4046D, IC6 40106D, IC7 4070D, IC8 4046D, IC9 4040D, Q1 THONKICONNNEW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

Commit message: finished routing, working on silkscreen
Connections:
- new net N$73: CCO1.SLEEVE, CCO2.SLEEVE, CCO3.SLEEVE, CCO4.SLEEVE, COMPLEX1.SLEEVE, COMPLEX2.SLEEVE
- net GND: no longer CCO1.SLEEVE, CCO2.SLEEVE, CCO3.SLEEVE, CCO4.SLEEVE, COMPLEX1.SLEEVE, COMPLEX2.SLEEVE
Changed lines of the file:
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@@
 <?xml version="1.0" encoding="utf-8"?>
 <!DOCTYPE eagle SYSTEM "eagle.dtd">
-<eagle version="9.0.1">
+<eagle version="8.5.2">
 <drawing>
 <settings>
@@
 <part name="COMPLEX1" library="MusicThingModular" deviceset="THONKICONN" device="NEW"/>
 <part name="COMPLEX2" library="MusicThingModular" deviceset="THONKICONN" device="NEW"/>
+<part name="GND70" library="supply1" deviceset="GND" device=""/>
 <part name="VCO1" library="MusicThingModular" deviceset="THONKICONN" device="NEW"/>
 <part name="VCO2" library="MusicThingModular" deviceset="THONKICONN" device="NEW"/>
@@
 <part name="GND74" library="supply1" library_urn="urn:adsk.eagle:library:371" deviceset="GND" device=""/>
 <part name="P+8" library="supply1" library_urn="urn:adsk.eagle:library:371" deviceset="V+" device=""/>
-<part name="GND70" library="supply1" deviceset="GND" device=""/>
 </parts>
 <sheets>
@@
 <wire x1="170.18" y1="58.42" x2="170.18" y2="55.88" width="0.1524" layer="91"/>
 <pinref part="C29" gate="G$1" pin="1"/>
-<junction x="157.48" y="58.42"/>
 </segment>
 </net>
@@
 <wire x1="157.48" y1="83.82" x2="170.18" y2="83.82" width="0.1524" layer="91"/>
 <wire x1="170.18" y1="83.82" x2="170.18" y2="81.28" width="0.1524" layer="91"/>
-<junction x="157.48" y="83.82"/>
 </segment>
 </net>
@@
 <wire x1="81.28" y1="243.84" x2="81.28" y2="238.76" width="0.1524" layer="91"/>
 </segment>
-<segment>
-<pinref part="CCO1" gate="G$1" pin="SLEEVE"/>
-<wire x1="345.44" y1="203.2" x2="337.82" y2="203.2" width="0.1524" layer="91"/>
-<wire x1="337.82" y1="203.2" x2="337.82" y2="198.12" width="0.1524" layer="91"/>
-<wire x1="337.82" y1="198.12" x2="365.76" y2="198.12" width="0.1524" layer="91"/>
-<wire x1="365.76" y1="198.12" x2="365.76" y2="180.34" width="0.1524" layer="91"/>
-<pinref part="CCO2" gate="G$1" pin="SLEEVE"/>
-<wire x1="365.76" y1="180.34" x2="365.76" y2="162.56" width="0.1524" layer="91"/>
-<wire x1="365.76" y1="162.56" x2="365.76" y2="144.78" width="0.1524" layer="91"/>
-<wire x1="365.76" y1="144.78" x2="365.76" y2="127" width="0.1524" layer="91"/>
-<wire x1="365.76" y1="127" x2="365.76" y2="109.22" width="0.1524" layer="91"/>
-<wire x1="365.76" y1="109.22" x2="365.76" y2="93.98" width="0.1524" layer="91"/>
-<wire x1="345.44" y1="185.42" x2="337.82" y2="185.42" width="0.1524" layer="91"/>
-<wire x1="337.82" y1="185.42" x2="337.82" y2="180.34" width="0.1524" layer="91"/>
-<wire x1="337.82" y1="180.34" x2="365.76" y2="180.34" width="0.1524" layer="91"/>
-<pinref part="CCO3" gate="G$1" pin="SLEEVE"/>
-<wire x1="345.44" y1="167.64" x2="337.82" y2="167.64" width="0.1524" layer="91"/>
-<wire x1="337.82" y1="167.64" x2="337.82" y2="162.56" width="0.1524" layer="91"/>
-<wire x1="337.82" y1="162.56" x2="365.76" y2="162.56" width="0.1524" layer="91"/>
-<pinref part="CCO4" gate="G$1" pin="SLEEVE"/>
-<wire x1="345.44" y1="149.86" x2="337.82" y2="149.86" width="0.1524" layer="91"/>
-<wire x1="337.82" y1="149.86" x2="337.82" y2="144.78" width="0.1524" layer="91"/>
-<wire x1="337.82" y1="144.78" x2="365.76" y2="144.78" width="0.1524" layer="91"/>
-<junction x="365.76" y="144.78"/>
-<junction x="365.76" y="162.56"/>
-<junction x="365.76" y="180.34"/>
-<wire x1="365.76" y1="127" x2="337.82" y2="127" width="0.1524" layer="91"/>
-<wire x1="337.82" y1="127" x2="337.82" y2="132.08" width="0.1524" layer="91"/>
-<pinref part="COMPLEX1" gate="G$1" pin="SLEEVE"/>
-<wire x1="337.82" y1="132.08" x2="345.44" y2="132.08" width="0.1524" layer="91"/>
-<pinref part="COMPLEX2" gate="G$1" pin="SLEEVE"/>
-<wire x1="345.44" y1="114.3" x2="337.82" y2="114.3" width="0.1524" layer="91"/>
-<wire x1="337.82" y1="114.3" x2="337.82" y2="109.22" width="0.1524" layer="91"/>
-<wire x1="337.82" y1="109.22" x2="365.76" y2="109.22" width="0.1524" layer="91"/>
-<junction x="365.76" y="109.22"/>
-<junction x="365.76" y="127"/>
-<pinref part="GND70" gate="1" pin="GND"/>
-</segment>
 </net>
 <net name="INV_C_IN" class="0">
@@
 <wire x1="345.44" y1="119.38" x2="332.74" y2="119.38" width="0.1524" layer="91"/>
 <label x="332.74" y="119.38" size="1.778" layer="95" rot="R180" xref="yes"/>
+</segment>
+</net>
+<net name="N$73" class="0">
+<segment>
+<pinref part="CCO1" gate="G$1" pin="SLEEVE"/>
+<wire x1="345.44" y1="203.2" x2="337.82" y2="203.2" width="0.1524" layer="91"/>
+<wire x1="337.82" y1="203.2" x2="337.82" y2="198.12" width="0.1524" layer="91"/>
+<wire x1="337.82" y1="198.12" x2="365.76" y2="198.12" width="0.1524" layer="91"/>
+<wire x1="365.76" y1="198.12" x2="365.76" y2="180.34" width="0.1524" layer="91"/>
+<pinref part="CCO2" gate="G$1" pin="SLEEVE"/>
+<wire x1="365.76" y1="180.34" x2="365.76" y2="162.56" width="0.1524" layer="91"/>
+<wire x1="365.76" y1="162.56" x2="365.76" y2="144.78" width="0.1524" layer="91"/>
+<wire x1="365.76" y1="144.78" x2="365.76" y2="127" width="0.1524" layer="91"/>
+<wire x1="365.76" y1="127" x2="365.76" y2="109.22" width="0.1524" layer="91"/>
+<wire x1="345.44" y1="185.42" x2="337.82" y2="185.42" width="0.1524" layer="91"/>
+<wire x1="337.82" y1="185.42" x2="337.82" y2="180.34" width="0.1524" layer="91"/>
+<wire x1="337.82" y1="180.34" x2="365.76" y2="180.34" width="0.1524" layer="91"/>
+<pinref part="CCO3" gate="G$1" pin="SLEEVE"/>
+<wire x1="345.44" y1="167.64" x2="337.82" y2="167.64" width="0.1524" layer="91"/>
+<wire x1="337.82" y1="167.64" x2="337.82" y2="162.56" width="0.1524" layer="91"/>
+<wire x1="337.82" y1="162.56" x2="365.76" y2="162.56" width="0.1524" layer="91"/>
+<pinref part="CCO4" gate="G$1" pin="SLEEVE"/>
+<wire x1="345.44" y1="149.86" x2="337.82" y2="149.86" width="0.1524" layer="91"/>
+<wire x1="337.82" y1="149.86" x2="337.82" y2="144.78" width="0.1524" layer="91"/>
+<wire x1="337.82" y1="144.78" x2="365.76" y2="144.78" width="0.1524" layer="91"/>
+<pinref part="COMPLEX1" gate="G$1" pin="SLEEVE"/>
+<wire x1="345.44" y1="132.08" x2="337.82" y2="132.08" width="0.1524" layer="91"/>
+<wire x1="337.82" y1="132.08" x2="337.82" y2="127" width="0.1524" layer="91"/>
+<wire x1="337.82" y1="127" x2="365.76" y2="127" width="0.1524" layer="91"/>
+<pinref part="COMPLEX2" gate="G$1" pin="SLEEVE"/>
+<wire x1="345.44" y1="114.3" x2="337.82" y2="114.3" width="0.1524" layer="91"/>
+<wire x1="337.82" y1="114.3" x2="337.82" y2="109.22" width="0.1524" layer="91"/>
+<wire x1="337.82" y1="109.22" x2="365.76" y2="109.22" width="0.1524" layer="91"/>
+<wire x1="365.76" y1="109.22" x2="365.76" y2="93.98" width="0.1524" layer="91"/>
+<pinref part="GND70" gate="1" pin="GND"/>
+<junction x="365.76" y="109.22"/>
+<junction x="365.76" y="127"/>
+<junction x="365.76" y="144.78"/>
+<junction x="365.76" y="162.56"/>
+<junction x="365.76" y="180.34"/>
 </segment>
 </net>
@@
 </sheet>
 </sheets>
-<errors>
-</errors>
 </schematic>
 </drawing>
