File: pcb_layouts/seamonster_smd/seamonster_buffered3.sch (EAGLE design)
At the start: 132 parts, among them IC1 7808DT, IC2 4051D, IC3 4051D, IC4 DG408DY, IC5 4046D, IC6 40106D, IC7 4070D, IC8 4046D, IC9 4040D, Q1 THONKICONNNEW, Q2 THONKICONNNEW, Q3 THONKICONNNEW, Q4 THONKICONNNEW, Q5 THONKICONNNEW, Q6 THONKICONNNEW, SW1 SPDT ON-ON, SW2 SPDT ON-ON, SW3 SPDT ON-ON, SW4 SPDT ON-ON, U1 TL084, U2 TL084, U3 TL084

Commit message: finished routing, working on silkscreen
Parts:
- removed C30, C31, C32, C33, C34, C35: (no value), SparkFun-Capacitors:CAP0805
- added C36, C37, C38, C39, C40, C41: (no value), SparkFun-Capacitors:10UF-25V-20%(PTH)
- added CVCO1, CVCO2: 1µF, SparkFun-Capacitors:CAP0805
- added U4: TL084D, linear:TL084D
- C23, C24: value 1µF -> 0.1µF
- IC2: value 4051D -> 40106D; device 40xx:4051D -> 40xx:40106D
- IC3: value 4051D -> 4040D; device 40xx:4051D -> 40xx:4040D
- IC4: value DG408DY -> 4051D; device maxim:DG408DY -> 40xx:4051D
- IC5: value 4046D -> 4051D; device 40xx:4046D -> 40xx:4051D
- IC6: value 40106D -> DG408DY; device 40xx:40106D -> maxim:DG408DY
- IC7: value 4070D -> 4046D; device 40xx:4070D -> 40xx:4046D
- IC9: value 4040D -> 4070D; device 40xx:4040D -> 40xx:4070D
- R1, R10, R11, R12, R13, R14, R2, R3, R4, R5, R6, R7, R8, R9: value (none) -> 270Ω
Connections:
- removed net Q1: IC9A.Q1, J1.2, Q1.TIP, R9.1
- new net N$61: IC3A.Q1, U3C.+IN
- new net Q1BUFFERED: J1.2, Q1.TIP, R9.1, U3C.-IN, U3C.OUT
- new net Q2BUFFERED: J2.2, Q2.TIP, R10.1, U3D.-IN, U3D.OUT
- new net Q3BUFFERED: J3.2, Q3.TIP, R11.1, U4A.-IN, U4A.OUT
- new net Q4BUFFERED: Q4.TIP, R12.1, U4B.-IN, U4B.OUT
- new net Q5BUFFERED: Q5.TIP, R13.1, U4C.-IN, U4C.OUT
- new net Q6BUFFERED: Q6.TIP, R14.1, U4D.-IN, U4D.OUT
- net A: now also IC4A.A, IC5A.A, IC6.A0; no longer IC2A.A, IC3A.A, IC4.A0
- net B: now also IC4A.B, IC5A.B, IC6.A1; no longer IC2A.B, IC3A.B, IC4.A1
- net C: now also IC4A.C, IC5A.C, IC6.A2; no longer IC2A.C, IC3A.C, IC4.A2
- net CCO1_BUFFERED: now also IC9A.I1; no longer IC7A.I1
- net CCO2_BUFFERED: now also IC9B.I1; no longer IC7B.I1
- net CCO3_BUFFERED: now also IC9C.I1; no longer IC7C.I1
- net CCO4_BUFFERED: now also IC9D.I1; no longer IC7D.I1
- net CV_OUT: now also IC4A.X; no longer IC3A.X
- net CV_OUT_BUFFERED: now also IC7A.VCOIN; no longer IC5A.VCOIN
- net GND: now also C23.2, C24.2, C36.-, C37.-, C38.-, C39.-, C40.-, C41.-, IC2P.VSS, IC3A.RES, IC3P.VSS, IC4A.INH, IC4P.GND, IC4P.VEE, IC5P.GND, IC5P.VEE, IC6.GND, IC7A.INH; no longer C30.2, C31.2, C32.2, C33.2, C34.2, C35.2, IC2A.INH, IC2P.GND, IC2P.VEE, IC3A.INH, IC3P.GND, IC3P.VEE, IC4.GND, IC5P.VSS, IC6P.VSS, IC9A.RES
- net INV_B_IN: now also IC2B.I; no longer IC6B.I
- net INV_B_OUT: now also IC2B.O; no longer IC6B.O
- net INV_C_IN: now also IC2C.I; no longer IC6C.I
- net INV_C_OUT: now also IC2C.O; no longer IC6C.O
- net INV_D_IN: now also IC2D.I; no longer IC6D.I
- net INV_D_OUT: now also IC2D.O; no longer IC6D.O
- net INV_E_IN: now also IC2E.I; no longer IC6E.I
- net INV_E_OUT: now also IC2E.O; no longer IC6E.O
- net MUX1: now also IC6.S1; no longer IC4.S1
- net MUX2: now also IC6.S2; no longer IC4.S2
- net MUX3: now also IC6.S3; no longer IC4.S3
- net MUX4: now also IC6.S4; no longer IC4.S4
- net MUX5: now also IC6.S5; no longer IC4.S5
- net MUX6: now also IC6.S6; no longer IC4.S6
- net MUX7: now also IC6.S7; no longer IC4.S7
- net MUX8: now also IC6.S8; no longer IC4.S8
- net N$1: now also IC6.D; no longer IC4.D
- net N$18: now also IC4A.X0; no longer IC3A.X0
- net N$19: now also IC5A.X0; no longer IC2A.X0
- net N$2: now also IC2A.I; no longer IC6A.I
- net N$20: now also IC5A.X1; no longer IC2A.X1
- net N$21: now also IC5A.X2; no longer IC2A.X2
- net N$22: now also IC5A.X3; no longer IC2A.X3
- net N$23: now also IC5A.X4; no longer IC2A.X4
- net N$24: now also IC5A.X5; no longer IC2A.X5
- net N$25: now also IC5A.X6; no longer IC2A.X6
- net N$26: now also IC5A.X7; no longer IC2A.X7
- net N$27: now also IC4A.X1; no longer IC3A.X1
- net N$28: now also IC4A.X2; no longer IC3A.X2
- net N$29: now also IC4A.X3; no longer IC3A.X3
- net N$3: now also C36.+; no longer C30.1
- net N$30: now also IC4A.X4; no longer IC3A.X4
- net N$31: now also IC4A.X5; no longer IC3A.X5
- net N$32: now also IC4A.X6; no longer IC3A.X6
- net N$33: now also IC4A.X7; no longer IC3A.X7
- net N$35: now also IC9A.O, IC9B.I0; no longer IC7A.O, IC7B.I0
- net N$36: now also IC9C.O, IC9D.I0; no longer IC7C.O, IC7D.I0
- net N$38: now also IC9B.O; no longer IC7B.O
- net N$39: now also IC9D.O; no longer IC7D.O
- net N$4: now also C37.+; no longer C31.1
- net N$40: now also IC7A.R2; no longer IC5A.R2
- net N$43: now also IC2A.O; no longer IC6A.O
- net N$44: now also CVCO1.1, IC7A.CX@1; no longer C23.1, IC5A.CX@1
- net N$45: now also CVCO1.2, IC7A.CX@2; no longer C23.2, IC5A.CX@2
- net N$48: now also CVCO2.1; no longer C24.1
- net N$49: now also CVCO2.2; no longer C24.2
- net N$5: now also C38.+; no longer C32.1
- net N$50: now also IC3A.P1; no longer IC9A.P1
- net N$6: now also C39.+; no longer C33.1
- net N$7: now also C40.+; no longer C34.1
- net N$75: now also IC7A.R1; no longer IC5A.R1
- net N$8: now also C41.+; no longer C35.1
- net Q2: now also IC3A.Q2, U3D.+IN; no longer IC9A.Q2, J2.2, Q2.TIP, R10.1
- net Q3: now also IC3A.Q3, U4A.+IN; no longer IC9A.Q3, J3.2, Q3.TIP, R11.1
- net Q4: now also IC3A.Q4, U4B.+IN; no longer IC9A.Q4, Q4.TIP, R12.1
- net Q5: now also IC3A.Q5, U4C.+IN; no longer IC9A.Q5, Q5.TIP, R13.1
- net Q6: now also IC3A.Q6, U4D.+IN; no longer IC9A.Q6, Q6.TIP, R14.1
- net V+: now also C23.1, IC6.EN, IC6.V+, U4P.V+; no longer IC4.EN, IC4.V+
- net V-: now also C24.1, IC6.V-, U4P.V-; no longer IC4.V-
- net VCC: now also IC2P.VDD, IC3P.VDD, IC4P.VCC, IC5A.X, IC5P.VCC; no longer IC2A.X, IC2P.VCC, IC3P.VCC, IC5P.VDD, IC6P.VDD
- net VCO1_OUT: now also IC7A.VCOOUT; no longer IC5A.VCOOUT
- net VCO2_OUT_BUFFERED: now also IC9A.I0, IC9C.I0; no longer IC7A.I0, IC7C.I0
Other:
- note added: "BUFFERED CV MULTIPLEXER SECTION This section uses a different multiplexing chip - the DG408DY to sequence bipolar CV signals upto +/-12V The signals patched into MUX inputs 1 thru 8 are sequenced and then buffered by U2D to create the final MUX output"
- note added: "BUFFERED CV OUTPUT SECTION IC3 is a 4051 8 way multiplexer chip, and is being used to select from one of eight potentiometers that are being used as voltage dividers and then being buffered by U2C to provide the final CV output"
- note added: "J1, J2 & J3 are jumpers that allow the assembler the option for normalized connection of the A, B & C clock signals to the Q1, Q2 & Q3 inputs to the multiplexer ICs"
- note added: "LED SEQUENCE INDICATOR SECTION Another 4051 multiplexer is being used to indicate the current step by lighting one of eight LEDs corresponding to the current step"
- moved on the sheet: CLOCK_IN, CLOCK_SELECT, IC7P, IC9P, LED10, LED11, LED12, LED13, LED14, LED9, Q1, Q2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

Commit message: worked on ai panel mockup, added TH capacitor optionally
Parts:
- removed C10, C12, C14, C7: 0.1µF, SparkFun-Capacitors:CAP0805
- removed C11, C13, C8, C9: 1µF, SparkFun-Capacitors:CAP0805
- removed C36, C37, C38, C39, C40, C41: (no value), SparkFun-Capacitors:10UF-25V-20%(PTH)
- added CCLK1, CCLK2, CCLK3, CCLK4, CCLK5, CCLK6: (no value), SparkFun-Capacitors:10UF-25V-20%(PTH)
- added CT1, CT2, CT3, CT4, CT5, CT6, CT7, CT8: (no value), SparkFun-Capacitors:CAP0805
- added CTH1, CTH2, CTH3, CTH4, CTH5, CTH6, CTH7, CTH8: (no value), SparkFun-Capacitors:CAP_POLPTH2
- U$2: value ALPHA_ROTARY_SWITCH -> CLOCK RATE SELECT
- renumbered C15 to CB3, C16 to CB4, C17 to CB5, C18 to CB12, C19 to CB13, C20 to CB6, C21 to CB7, C22 to CB8, C23 to CB16, C24 to CB17, C25 to CB18, C26 to CB19, C27 to CB9, C28 to CB14, C29 to CB15, C3 to CB1, C4 to CB2, C5 to CB10, C6 to CB11, CVCO1 to CT9, CVCO2 to CT10
Connections:
- net GND: now also CCLK1.-, CCLK2.-, CCLK3.-, CCLK4.-, CCLK5.-, CCLK6.-, CT1.2, CT2.2, CT3.2, CT4.2, CT5.2, CT6.2, CT7.2, CT8.2, CTH1.-, CTH2.-, CTH3.-, CTH4.-, CTH5.-, CTH6.-, CTH7.-, CTH8.-; no longer C10.2, C11.2, C12.2, C13.2, C14.2, C36.-, C37.-, C38.-, C39.-, C40.-, C41.-, C7.2, C8.2, C9.2
- net N$3: now also CCLK1.+; no longer C36.+
- net N$4: now also CCLK2.+; no longer C37.+
- net N$47: now also CT2.1, CTH2.+; no longer C7.1
- net N$5: now also CCLK3.+; no longer C38.+
- net N$52: now also CT1.1, CTH1.+; no longer C8.1
- net N$55: now also CT4.1, CTH4.+; no longer C10.1
- net N$56: now also CT3.1, CTH3.+; no longer C9.1
- net N$59: now also CT6.1, CTH6.+; no longer C12.1
- net N$6: now also CCLK4.+; no longer C39.+
- net N$60: now also CT5.1, CTH5.+; no longer C11.1
- net N$63: now also CT8.1, CTH8.+; no longer C14.1
- net N$64: now also CT7.1, CTH7.+; no longer C13.1
- net N$7: now also CCLK5.+; no longer C40.+
- net N$8: now also CCLK6.+; no longer C41.+

Commit message: smd mk1 routing complete
Connections:
- net VCO1_OUT_BUFFERED: now also IC9A.I0
- net VCO2_OUT_BUFFERED: no longer IC9A.I0
Changed lines of the file:
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@@
 <setting verticaltext="up"/>
 </settings>
-<grid distance="0.1" unitdist="inch" unit="inch" style="lines" multiple="1" display="yes" altdistance="0.01" altunitdist="inch" altunit="inch"/>
+<grid distance="0.1" unitdist="inch" unit="inch" style="lines" multiple="1" display="no" altdistance="0.01" altunitdist="inch" altunit="inch"/>
 <layers>
 <layer number="1" name="Top" color="4" fill="1" visible="no" active="no"/>
@@
 <label x="157.48" y="116.84" size="1.778" layer="95" rot="R180" xref="yes"/>
 </segment>
+</net>
+<net name="VCO1_OUT_BUFFERED" class="0">
 <segment>
 <pinref part="IC9" gate="A" pin="I0"/>
-<wire x1="175.26" y1="215.9" x2="167.64" y2="215.9" width="0.1524" layer="91"/>
-<wire x1="167.64" y1="215.9" x2="167.64" y2="223.52" width="0.1524" layer="91"/>
-<wire x1="167.64" y1="223.52" x2="160.02" y2="223.52" width="0.1524" layer="91"/>
-<label x="160.02" y="223.52" size="1.778" layer="95" rot="R180" xref="yes"/>
-</segment>
-</net>
+<wire x1="175.26" y1="215.9" x2="162.56" y2="215.9" width="0.1524" layer="91"/>
+<wire x1="162.56" y1="215.9" x2="162.56" y2="226.06" width="0.1524" layer="91"/>
+<wire x1="162.56" y1="226.06" x2="154.94" y2="226.06" width="0.1524" layer="91"/>
+<label x="154.94" y="226.06" size="1.778" layer="95" rot="R180" xref="yes"/>
+</segment>
+</net>
